Commit message: some world | urdf | launch files update

File: driverless_ws/src/driverless_package/urdf/test.urdf (robot description, URDF)
Before this commit: robot robot_arm, 2 links, 1 joints
Links:
- removed link link_01
- added link body; visual box size=0.58 0.2 0.01
- added link camera_depth_optical_frame; visual box size=.001 .001 .001
- added link imu; visual box size=.01 .01 .01
- added link left_front_steering; visual box size=.001 .001 .001
- added link left_front_wheel; visual cylinder length=0.043 radius=0.054
- added link left_rear_wheel; visual cylinder length=0.043 radius=0.054
- added link lidar; visual cylinder length=0.020 radius=0.039
- added link realsense; visual box size=0.015 0.139 0.051
- added link right_front_steering; visual box size=.001 .001 .001
- added link right_front_wheel; visual cylinder length=0.043 radius=0.054
- added link right_rear_wheel; visual cylinder length=0.043 radius=0.054
- link base_link: mass 0.2 -> None; geometry visual box size=.001 .001 .001
Joints:
- removed joint base_link__link_01
- added joint base_link_to_body: type revolute, parent base_link, child body, origin xyz=0 0 0.054, axis 0 1 0, limit lower=-0.065 upper=0.065 effort=1000 velocity=1000
- added joint base_link_to_left_front_steering: type revolute, parent base_link, child left_front_steering, origin xyz=0.326 0.125 0.054, axis 0 0 1, limit lower=-0.87 upper=0.87 effort=1000 velocity=1000
- added joint base_link_to_right_front_steering: type revolute, parent base_link, child right_front_steering, origin xyz=0.326 -0.125 0.054, axis 0 0 1, limit lower=-0.87 upper=0.87 effort=1000 velocity=1000
- added joint body_to_camera_depth_optical_frame: type revolute, parent body, child camera_depth_optical_frame, origin xyz=0.226 0.04 0.177 rpy=-1.57079 0 -1.57079, axis 0 0 1, limit lower=-0.001 upper=0.001 effort=1000 velocity=1000
- added joint body_to_imu: type fixed, parent body, child imu, origin xyz=0.236 0 0.082
- added joint body_to_left_rear_wheel: type continuous, parent body, child left_rear_wheel, origin xyz=0 0.125 0.0, axis 0 1 0
- added joint body_to_lidar: type fixed, parent body, child lidar, origin xyz=0.339 0 0.107 rpy=0 0 3.1415926
- added joint body_to_realsense: type fixed, parent body, child realsense, origin xyz=0.226 -0.044 0.177
- added joint body_to_right_rear_wheel: type continuous, parent body, child right_rear_wheel, origin xyz=0 -0.125 0.0, axis 0 1 0
- added joint left_front_steering_to_left_front_wheel: type continuous, parent left_front_steering, child left_front_wheel, origin xyz=0.0 0.0 0.0, axis 0 1 0
- added joint right_front_steering_to_right_front_wheel: type continuous, parent right_front_steering, child right_front_wheel, origin xyz=0.0 0.0 0.0, axis 0 1 0
